File: rsttl.kicad_pcb (KiCad board)
At the start: 2 copper layers, 83.2 x 32 mm, 18 parts, among them J1 DB9_Male, J2 7-20V Ext, J3 TTL Data, 5V, J4 5V Ext SW, J5 DB9_Female, U1 L7805, U2 MAX232

Commit message: Try new layour
Parts:
- moved J4 9.80 mm to (142.4, 91.7)
- moved C3 2.30 mm to (128.1, 95.4)
- moved C1 2.30 mm to (114.4, 98.0)
- moved U1 2.30 mm to (121.3, 96.6)
- moved J2 1.21 mm to (112.0, 92.4)
- moved U2 0.95 mm to (130.7, 110.5)
- moved C6 0.95 mm to (126.1, 106.6)
- moved C4 0.95 mm to (132.1, 98.5)
- moved C2 0.95 mm to (132.1, 115.2)
- moved C5 0.95 mm to (139.6, 115.2)
- moved C7 0.95 mm to (147.1, 115.2)
- moved J3 0.50 mm to (106.4, 92.4)
- moved D1 0.40 mm to (105.8, 114.6)
- moved D2 0.40 mm to (111.6, 114.6)
- moved R1 0.40 mm to (105.8, 108.9)
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Changed lines of the file:
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@@
   (general
     (thickness 1.6)
-    (drawings 9)
+    (drawings 13)
     (tracks 140)
     (zones 0)
@@
   )
   (layers
-    (0 F.Cu signal)
-    (31 B.Cu signal)
+    (0 F.Cu signal hide)
+    (31 B.Cu signal hide)
     (32 B.Adhes user hide)
     (33 F.Adhes user hide)
@@
   )
   (module Capacitor_SMD:C_1206_3216Metric (layer F.Cu)
-    (at 114.4 95.7)
+    (at 114.4 98)
     (descr "Capacitor SMD 1206 (3216 Metric), square (rectangular) end terminal, IPC_7351 nominal, (Body size source: http://www.tortai-tech.com/upload/download/2011102023233369053.pdf), generated with kicad-footprint-generator")
     (tags capacitor)
@@
   )
   (module Capacitor_SMD:C_1210_3225Metric (layer F.Cu)
-    (at 131.8 116.1)
+    (at 132.1 115.2)
     (descr "Capacitor SMD 1210 (3225 Metric), square (rectangular) end terminal, IPC_7351 nominal, (Body size source: http://www.tortai-tech.com/upload/download/2011102023233369053.pdf), generated with kicad-footprint-generator")
     (tags capacitor)
@@
   )
   (module Capacitor_SMD:C_0805_2012Metric (layer F.Cu)
-    (at 128.1 93.1 90)
+    (at 128.1 95.4 90)
     (descr "Capacitor SMD 0805 (2012 Metric), square (rectangular) end terminal, IPC_7351 nominal, (Body size source: https://docs.google.com/spreadsheets/d/1BsfQQcO9C6DZCsRaXUlFlo91Tg2WpOkGARC1WS5S8t0/edit?usp=sharing), generated with kicad-footprint-generator")
     (tags capacitor)
@@
   )
   (module Capacitor_SMD:C_1210_3225Metric (layer F.Cu)
-    (at 131.8 99.4)
+    (at 132.1 98.5)
     (descr "Capacitor SMD 1210 (3225 Metric), square (rectangular) end terminal, IPC_7351 nominal, (Body size source: http://www.tortai-tech.com/upload/download/2011102023233369053.pdf), generated with kicad-footprint-generator")
     (tags capacitor)
@@
   )
   (module Capacitor_SMD:C_1210_3225Metric (layer F.Cu)
-    (at 139.3 116.1)
+    (at 139.6 115.2)
     (descr "Capacitor SMD 1210 (3225 Metric), square (rectangular) end terminal, IPC_7351 nominal, (Body size source: http://www.tortai-tech.com/upload/download/2011102023233369053.pdf), generated with kicad-footprint-generator")
     (tags capacitor)
@@
   )
   (module Capacitor_SMD:C_1210_3225Metric (layer F.Cu)
-    (at 125.8 107.5 90)
+    (at 126.1 106.6 90)
     (descr "Capacitor SMD 1210 (3225 Metric), square (rectangular) end terminal, IPC_7351 nominal, (Body size source: http://www.tortai-tech.com/upload/download/2011102023233369053.pdf), generated with kicad-footprint-generator")
     (tags capacitor)
@@
   )
   (module Capacitor_SMD:C_1210_3225Metric (layer F.Cu)
-    (at 146.8 116.1 180)
+    (at 147.1 115.2 180)
     (descr "Capacitor SMD 1210 (3225 Metric), square (rectangular) end terminal, IPC_7351 nominal, (Body size source: http://www.tortai-tech.com/upload/download/2011102023233369053.pdf), generated with kicad-footprint-generator")
     (tags capacitor)
@@
   )
   (module LED_SMD:LED_1210_3225Metric (layer F.Cu)
-    (at 105.8 115 90)
+    (at 105.8 114.6 90)
     (descr "LED SMD 1210 (3225 Metric), square (rectangular) end terminal, IPC_7351 nominal, (Body size source: http://www.tortai-tech.com/upload/download/2011102023233369053.pdf), generated with kicad-footprint-generator")
     (tags diode)
@@
   )
   (module LED_SMD:LED_1210_3225Metric (layer F.Cu)
-    (at 111.6 115 90)
+    (at 111.6 114.6 90)
     (descr "LED SMD 1210 (3225 Metric), square (rectangular) end terminal, IPC_7351 nominal, (Body size source: http://www.tortai-tech.com/upload/download/2011102023233369053.pdf), generated with kicad-footprint-generator")
     (tags diode)
@@
   )
   (module Connector_PinHeader_2.54mm:PinHeader_1x02_P2.54mm_Vertical (layer F.Cu)
-    (at 113.1 91.9 90)
+    (at 112 92.4 90)
     (descr "Through hole straight pin header, 1x02, 2.54mm pitch, single row")
     (tags "Through hole pin header THT 1x02 2.54mm single row")
@@
   )
   (module Connector_PinHeader_2.54mm:PinHeader_1x04_P2.54mm_Vertical (layer F.Cu)
-    (at 106.4 91.9)
+    (at 106.4 92.4)
     (descr "Through hole straight pin header, 1x04, 2.54mm pitch, single row")
     (tags "Through hole pin header THT 1x04 2.54mm single row")
@@
   )
   (module Connector_PinHeader_2.54mm:PinHeader_1x02_P2.54mm_Vertical (layer F.Cu)
-    (at 132.6 92)
+    (at 142.4 91.7)
     (descr "Through hole straight pin header, 1x02, 2.54mm pitch, single row")
     (tags "Through hole pin header THT 1x02 2.54mm single row")
@@
   )
   (module Resistor_SMD:R_1210_3225Metric (layer F.Cu)
-    (at 105.8 109.3 270)
+    (at 105.8 108.9 270)
     (descr "Resistor SMD 1210 (3225 Metric), square (rectangular) end terminal, IPC_7351 nominal, (Body size source: http://www.tortai-tech.com/upload/download/2011102023233369053.pdf), generated with kicad-footprint-generator")
     (tags resistor)
@@
   )
   (module Resistor_SMD:R_1210_3225Metric (layer F.Cu)
-    (at 111.6 109.3 270)
+    (at 111.6 108.9 270)
     (descr "Resistor SMD 1210 (3225 Metric), square (rectangular) end terminal, IPC_7351 nominal, (Body size source: http://www.tortai-tech.com/upload/download/2011102023233369053.pdf), generated with kicad-footprint-generator")
     (tags resistor)
@@
   )
   (module Package_TO_SOT_SMD:TO-252-2 (layer F.Cu)
-    (at 121.3 94.3 90)
+    (at 121.3 96.6 90)
     (descr "TO-252 / DPAK SMD package, http://www.infineon.com/cms/en/product/packages/PG-TO252/PG-TO252-3-1/")
     (tags "DPAK TO-252 DPAK-3 TO-252-3 SOT-428")
@@
   )
   (module Package_DIP:DIP-16_W7.62mm_LongPads (layer F.Cu)
-    (at 130.42 111.4 90)
+    (at 130.72 110.5 90)
     (descr "16-lead though-hole mounted DIP package, row spacing 7.62 mm (300 mils), LongPads")
     (tags "THT DIP DIL PDIP 2.54mm 7.62mm 300mil LongPads")
@@
     )
   )
+  (gr_line (start 88.4 91) (end 165.6 91) (layer Margin) (width 0.15))
+  (gr_line (start 88.4 117) (end 88.4 91) (layer Margin) (width 0.15))
+  (gr_line (start 165.6 117) (end 88.4 117) (layer Margin) (width 0.15))
+  (gr_line (start 165.6 91) (end 165.6 117) (layer Margin) (width 0.15))
   (gr_text rev.A (at 163.7 104 90) (layer B.SilkS)
     (effects (font (size 3 3) (thickness 0.3)) (justify mirror))
   )
-  (gr_text Tx (at 105.8 118.5) (layer F.SilkS)
+  (gr_text Tx (at 105.8 118.1) (layer F.SilkS)
     (effects (font (size 1 1) (thickness 0.15)))
   )
-  (gr_text Rx (at 111.6 118.5) (layer F.SilkS)
+  (gr_text Rx (at 111.6 118.1) (layer F.SilkS)
     (effects (font (size 1 1) (thickness 0.15)))
   )
-  (gr_text Gnd (at 103.3 94.5) (layer F.SilkS)
+  (gr_text Gnd (at 103.3 95) (layer F.SilkS)
     (effects (font (size 1 1) (thickness 0.15)))
   )
-  (gr_text 5V (at 103.2 91.9) (layer F.SilkS)
+  (gr_text 5V (at 103.3 92.4) (layer F.SilkS)
     (effects (font (size 1 1) (thickness 0.15)))
   )

Commit message: Layout revA
Parts:
- moved J4 12.2 mm to (130.3, 92.4), turned to 90 degrees
- moved C3 3.29 mm to (127.2, 98.6)
- moved C4 1.20 mm to (133.3, 98.4)
- moved C6 0.90 mm to (126.1, 107.5)
Routing:
- net GND: track 35.0 -> 47.8 mm, vias 5 -> 3
- net +5V: track 49.8 -> 51.7 mm
- net Net-(C6-Pad1): track 8.71 -> 10.6 mm
- net VCC: track 11.7 -> 13.5 mm
- net Net-(J5-Pad2): track 15.9 -> 14.8 mm
- net Net-(J1-Pad2): track 70.2 -> 70.7 mm
- net Net-(C3-Pad1): track 13.5 -> 12.9 mm
Other:
- rule trace_min: 0.5 -> 0.2

Commit message: Add symbols
Parts:
- added REF**: OSHW-Logo2_7.3x6mm_SilkScreen, Symbol:OSHW-Logo2_7.3x6mm_SilkScreen, F.Cu at (121.1, 115.0)
- added REF**: KiCad-Logo2_5mm_SilkScreen, Symbol:KiCad-Logo2_5mm_SilkScreen, F.Cu at (143.7, 92.5)
