File: rsttl.kicad_pcb (KiCad board)
At the start: 2 copper layers, 83.2 x 32 mm, 20 parts, among them J1 DB9_Male, J2 7-20V Ext, J3 TTL Data, 5V, J4 5V Ext SW, J5 DB9_Female, U1 L7805, U2 MAX232

Commit message: 'Fixes'
Routing:
- net Net-(C5-Pad2): track 4.11 -> 5.15 mm
- net GND: track 47.8 -> 46.8 mm
- net Net-(C2-Pad2): track 6.01 -> 6.94 mm
- net Net-(J1-Pad3): track 57.1 -> 57.7 mm
- net Net-(C7-Pad2): track 5.91 -> 6.51 mm
Changed lines of the file:
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@@
-(kicad_pcb (version 20171130) (host pcbnew "(5.1.4)-1")
+(kicad_pcb (version 20171130) (host pcbnew "(5.1.5)-3")
   (general
     (thickness 1.6)
     (drawings 13)
-    (tracks 145)
+    (tracks 146)
     (zones 0)
     (modules 20)
@@
   (segment (start 132.54 105.9) (end 125.6 105.9) (width 0.5) (layer F.Cu) (net 2))
   (segment (start 132.96 103.78) (end 132.96 102.08) (width 0.5) (layer F.Cu) (net 2))
-  (via (at 151.4 116.4) (size 0.8) (drill 0.4) (layers F.Cu B.Cu) (net 2))
   (via (at 102.6 116.4) (size 0.8) (drill 0.4) (layers F.Cu B.Cu) (net 2))
   (via (at 114.8 116.4) (size 0.8) (drill 0.4) (layers F.Cu B.Cu) (net 2))
   (segment (start 102.6 116.4) (end 105.6 116.4) (width 0.5) (layer F.Cu) (net 2))
   (segment (start 111.6 116.4) (end 114.8 116.4) (width 0.5) (layer F.Cu) (net 2))
-  (segment (start 150.834315 116.4) (end 150.534315 116.1) (width 0.5) (layer F.Cu) (net 2))
-  (segment (start 151.4 116.4) (end 150.834315 116.4) (width 0.5) (layer F.Cu) (net 2))
-  (segment (start 150.534315 116.1) (end 148.3 116.1) (width 0.5) (layer F.Cu) (net 2))
   (segment (start 114.54 93.602081) (end 115.8 94.862081) (width 1) (layer F.Cu) (net 2))
   (segment (start 114.54 92.4) (end 114.54 93.602081) (width 1) (layer F.Cu) (net 2))
@@
   (segment (start 125.6625 95.5) (end 116.437919 95.5) (width 1) (layer F.Cu) (net 2))
   (segment (start 125.6625 95.5) (end 121.5 95.5) (width 1) (layer F.Cu) (net 2))
+  (via (at 150.500002 115.2) (size 0.8) (drill 0.4) (layers F.Cu B.Cu) (net 2))
+  (segment (start 148.3 115.2) (end 150.500002 115.2) (width 0.5) (layer F.Cu) (net 2))
   (segment (start 130.42 111.4) (end 130.42 115.98) (width 0.5) (layer F.Cu) (net 3))
-  (segment (start 135.5 114.525) (end 135.5 113.1) (width 0.5) (layer F.Cu) (net 4))
-  (segment (start 135.5 113.1) (end 135.5 111.4) (width 0.5) (layer F.Cu) (net 4))
-  (segment (start 135.5 114.525) (end 135.5 115.1) (width 0.5) (layer F.Cu) (net 4))
-  (segment (start 135.5 115.1) (end 134.5 116.1) (width 0.5) (layer F.Cu) (net 4))
-  (segment (start 134.5 116.1) (end 133.6 116.1) (width 0.5) (layer F.Cu) (net 4))
+  (segment (start 135.8 112.8) (end 135.8 110.6) (width 0.5) (layer F.Cu) (net 4))
+  (segment (start 135.8 114.8) (end 135.8 112.8) (width 0.5) (layer F.Cu) (net 4))
+  (segment (start 133.6 116.1) (end 134.5 116.1) (width 0.5) (layer F.Cu) (net 4))
+  (segment (start 134.5 116.1) (end 135.8 114.8) (width 0.5) (layer F.Cu) (net 4))
   (segment (start 123.58 100.8) (end 125.9 100.8) (width 1) (layer F.Cu) (net 5))
   (segment (start 125.9 100.8) (end 127.2 99.5) (width 1) (layer F.Cu) (net 5))
@@
   (segment (start 131.9 96.3) (end 132.8 95.4) (width 0.5) (layer F.Cu) (net 6))
   (segment (start 132.8 95.4) (end 132.8 92.4) (width 0.5) (layer F.Cu) (net 6))
-  (segment (start 138.04 111.4) (end 138.04 115.46) (width 0.5) (layer F.Cu) (net 7))
-  (segment (start 140.58 113.1) (end 140.6 113.12) (width 0.5) (layer F.Cu) (net 8))
-  (segment (start 140.58 111.4) (end 140.58 113.1) (width 0.5) (layer F.Cu) (net 8))
-  (segment (start 140.6 113.12) (end 140.6 115.5) (width 0.5) (layer F.Cu) (net 8))
+  (segment (start 138.3 115.2) (end 138.04 115.46) (width 0.5) (layer F.Cu) (net 7))
+  (segment (start 138.04 111.4) (end 138.3 111.66) (width 0.5) (layer F.Cu) (net 7))
+  (segment (start 138.3 111.66) (end 138.3 115.2) (width 0.5) (layer F.Cu) (net 7))
+  (segment (start 141 115.1) (end 140.6 115.5) (width 0.5) (layer F.Cu) (net 8))
+  (segment (start 140.8 110.6) (end 141 110.8) (width 0.5) (layer F.Cu) (net 8))
+  (segment (start 141 110.8) (end 141 115.1) (width 0.5) (layer F.Cu) (net 8))
   (segment (start 132.96 111.4) (end 132.96 109.7) (width 0.5) (layer F.Cu) (net 9))
   (segment (start 133.26 108.8) (end 132.46 108) (width 0.5) (layer F.Cu) (net 9))
@@
   (segment (start 129 108) (end 128.1 108.9) (width 0.5) (layer F.Cu) (net 9))
   (segment (start 128.1 108.9) (end 126.8 108.9) (width 0.5) (layer F.Cu) (net 9))
-  (segment (start 143.12 113.1) (end 143.1 113.12) (width 0.5) (layer F.Cu) (net 10))
-  (segment (start 143.12 111.4) (end 143.12 113.1) (width 0.5) (layer F.Cu) (net 10))
-  (segment (start 143.1 113.12) (end 143.1 114.8) (width 0.5) (layer F.Cu) (net 10))
-  (segment (start 143.1 114.8) (end 144.3 116) (width 0.5) (layer F.Cu) (net 10))
-  (segment (start 144.3 116) (end 145.1 116) (width 0.5) (layer F.Cu) (net 10))
+  (segment (start 144.4 115.4) (end 145.6 115.4) (width 0.5) (layer F.Cu) (net 10))
+  (segment (start 143.5 114.5) (end 144.4 115.4) (width 0.5) (layer F.Cu) (net 10))
+  (segment (start 143.4 110.5) (end 143.5 110.6) (width 0.5) (layer F.Cu) (net 10))
+  (segment (start 143.5 110.6) (end 143.5 114.5) (width 0.5) (layer F.Cu) (net 10))
   (segment (start 105.8 110.7) (end 105.8 113.5) (width 0.5) (layer F.Cu) (net 11))
   (segment (start 111.6 110.7) (end 111.6 111.425) (width 0.5) (layer F.Cu) (net 12))
@@
   (segment (start 145.66 102.08) (end 143.18 99.6) (width 0.5) (layer B.Cu) (net 13))
   (segment (start 145.66 103.78) (end 145.66 102.08) (width 0.5) (layer B.Cu) (net 13))
-  (segment (start 100.86 104.04) (end 100.86 104.06) (width 0.5) (layer F.Cu) (net 13))
-  (segment (start 100.86 104.06) (end 104.7 107.9) (width 0.5) (layer F.Cu) (net 13))
   (segment (start 143.18 99.6) (end 106.4 99.6) (width 0.5) (layer B.Cu) (net 13))
   (segment (start 100.86 104.04) (end 98.6 104.04) (width 0.5) (layer F.Cu) (net 13))
-  (segment (start 105.3 99.6) (end 106.4 99.6) (width 0.5) (layer F.Cu) (net 13))
-  (segment (start 105.3 99.6) (end 100.86 104.04) (width 0.5) (layer F.Cu) (net 13))
+  (segment (start 106.4 100) (end 106.4 99.6) (width 0.5) (layer F.Cu) (net 13))
+  (segment (start 106.5 100.1) (end 106.4 100) (width 0.5) (layer F.Cu) (net 13))
+  (segment (start 100.86 104.04) (end 104.8 100.1) (width 0.5) (layer F.Cu) (net 13))
+  (segment (start 104.8 100.1) (end 106.5 100.1) (width 0.5) (layer F.Cu) (net 13))
+  (segment (start 104 107.5) (end 104.9 107.5) (width 0.5) (layer F.Cu) (net 13))
+  (segment (start 100.86 104.04) (end 100.86 104.36) (width 0.5) (layer F.Cu) (net 13))
+  (segment (start 100.86 104.36) (end 104 107.5) (width 0.5) (layer F.Cu) (net 13))
   (segment (start 148.2 103.78) (end 148.2 102.08) (width 0.5) (layer B.Cu) (net 14))
   (segment (start 111.6 107.9) (end 111.6 107.175) (width 0.5) (layer F.Cu) (net 14))

Commit message: Update
Parts:
- C1: footprint Capacitor_SMD:C_1206_3216Metric -> Capacitor_SMD:C_1210_3225Metric
- C3: footprint Capacitor_SMD:C_0805_2012Metric -> Capacitor_SMD:C_1210_3225Metric
- D1, D2: footprint LED_SMD:LED_1210_3225Metric -> LED_SMD:LED_0805_2012Metric
- moved C3 0.60 mm to (127.8, 98.6)
- moved C4 0.20 mm to (133.5, 98.4)
Routing:
- net Net-(C3-Pad1): track 12.9 -> 13.9 mm
- net GND: track 46.8 -> 47.5 mm, vias 3 -> 2
