File: rsttl.sch (KiCad schematic (older format))
At the start: 18 parts, among them J1 DB9_Male, J2 7-20V Ext, J3 TTL Data, 5V, J4 5V Ext SW, J5 DB9_Female, U1 L7805, U2 MAX232

Commit message: Update
Parts:
- C1: footprint Capacitor_SMD:C_1206_3216Metric -> Capacitor_SMD:C_1210_3225Metric
- C3: footprint Capacitor_SMD:C_0805_2012Metric -> Capacitor_SMD:C_1210_3225Metric
- D1, D2: footprint LED_SMD:LED_1210_3225Metric -> LED_SMD:LED_0805_2012Metric
Changed lines of the file:
@@
 EESchema Schematic File Version 4
-LIBS:rsttl-cache
 EELAYER 30 0
 EELAYER END
@@
 F 0 "D1" V 5046 6982 50  0000 R CNN
 F 1 "LED_Small" V 4955 6982 50  0000 R CNN
-F 2 "LED_SMD:LED_1210_3225Metric" V 5000 7050 50  0001 C CNN
+F 2 "LED_SMD:LED_0805_2012Metric" V 5000 7050 50  0001 C CNN
 F 3 "~" V 5000 7050 50  0001 C CNN
 	1    5000 7050
@@
 F 0 "D2" V 5546 6982 50  0000 R CNN
 F 1 "LED_Small" V 5455 6982 50  0000 R CNN
-F 2 "LED_SMD:LED_1210_3225Metric" V 5500 7050 50  0001 C CNN
+F 2 "LED_SMD:LED_0805_2012Metric" V 5500 7050 50  0001 C CNN
 F 3 "~" V 5500 7050 50  0001 C CNN
 	1    5500 7050
@@
 F 0 "C1" H 4968 1996 50  0000 L CNN
 F 1 "0.33uF" H 4968 1905 50  0000 L CNN
-F 2 "Capacitor_SMD:C_1206_3216Metric" H 4888 1800 50  0001 C CNN
+F 2 "Capacitor_SMD:C_1210_3225Metric" H 4888 1800 50  0001 C CNN
 F 3 "~" H 4850 1950 50  0001 C CNN
 	1    4850 1950
@@
 F 0 "C3" H 7218 2046 50  0000 L CNN
 F 1 "0.1F" H 7218 1955 50  0000 L CNN
-F 2 "Capacitor_SMD:C_0805_2012Metric" H 7138 1850 50  0001 C CNN
+F 2 "Capacitor_SMD:C_1210_3225Metric" H 7138 1850 50  0001 C CNN
 F 3 "~" H 7100 2000 50  0001 C CNN
 	1    7100 2000
