File: rsttl.sch (KiCad schematic (older format))
At the start: 18 parts, among them J1 DB9_Male, J2 7-20V Ext, J3 TTL Data, 5V, J4 5V Ext SW, J5 DB9_Female, U1 L7805, U2 MAX232

Commit message: Rev.B
Parts:
- removed J4: 5V Ext SW, Connector_PinHeader_2.54mm:PinHeader_1x02_P2.54mm_Vertical, symbol Connector_Generic:Conn_01x02
- C1: footprint Capacitor_SMD:C_1210_3225Metric -> Capacitor_SMD:C_1210_3225Metric_Pad1.42x2.65mm_HandSolder
- C2, C4, C5, C6, C7: footprint Capacitor_SMD:C_1210_3225Metric -> Capacitor_SMD:C_0805_2012Metric_Pad1.15x1.40mm_HandSolder
- C3: value 0.1F -> 0.1uF; footprint Capacitor_SMD:C_1210_3225Metric -> Capacitor_SMD:C_1210_3225Metric_Pad1.42x2.65mm_HandSolder
- J3: footprint Connector_PinHeader_2.54mm:PinHeader_1x04_P2.54mm_Vertical -> Connector_PinHeader_2.54mm:PinHeader_1x06_P2.54mm_Vertical; symbol Connector_Generic:Conn_01x04 -> Connector_Generic:Conn_01x06
- R1, R2: footprint Resistor_SMD:R_1210_3225Metric -> Resistor_SMD:R_0805_2012Metric_Pad1.15x1.40mm_HandSolder
- U1: value L7805 -> NCP1117; footprint Package_TO_SOT_SMD:TO-252-2 -> Package_TO_SOT_SMD:SOT-223-3_TabPin2; symbol Regulator_Linear:L7805 -> Regulator_Linear:NCP1117-5.0_SOT223
- U2: footprint Package_DIP:DIP-16_W7.62mm_LongPads -> Package_SO:SOP-16_4.55x10.3mm_P1.27mm
Connections:
- wire segments 73 -> 78
Other:
- moved on the sheet: D1, D2
